File: OFMBearBoard/OFMBearBoard.kicad_sch (KiCad schematic)
At the start: 11 parts, among them J1 X Motor, J2 Y Motor, J3 Z Motor, J4 LED, J5 5V, U1 ULN2003APG, U2 ULN2003APG

Commit message: Fixed IC aligment and capacitor size
Fixed IC aligment and capacitor size
Parts:
- C1, C2: footprint Capacitor_THT:C_Disc_D3.0mm_W2.0mm_P2.50mm -> Capacitor_THT:C_Disc_D9.0mm_W2.5mm_P5.00mm
Changed lines of the file:
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@@
 			)
 		)
-		(property "Footprint" "Capacitor_THT:C_Disc_D3.0mm_W2.0mm_P2.50mm"
+		(property "Footprint" "Capacitor_THT:C_Disc_D9.0mm_W2.5mm_P5.00mm"
 			(at 147.6248 22.86 0)
 			(effects
@@
 			)
 		)
-		(property "Footprint" "Capacitor_THT:C_Disc_D3.0mm_W2.0mm_P2.50mm"
+		(property "Footprint" "Capacitor_THT:C_Disc_D9.0mm_W2.5mm_P5.00mm"
 			(at 147.6248 62.23 0)
 			(effects
